Commit message: Added a ROS service for object detection via machine vision using the realsense ROS2 wrapper, alsos added a protopyte motions package for adding in future robot motions

File: ri_seaweed_ws/src/robot_description/gripper_support/urdf/gripper.xacro (robot description, xacro)
@@ -262,4 +262,11 @@
   <child link="claw_body_r_1"/>
 </joint>
+<!-- Transfer from camera to gripper base -->
+<link name="camera_frame"></link>
+<joint name="gripper-base_link_to_camera_joint" type="fixed">
+  <parent link="gripper-base_link"/>
+  <child link="camera_frame"/>
+  <origin xyz="-0.17 0.033 -0.033" rpy="3.14159265 0 0"/>
+</joint>
 </xacro:macro>
 </robot>

Commit message: Fixed gripper orientation

File: ri_seaweed_ws/src/robot_description/gripper_support/urdf/gripper.xacro (robot description, xacro)
@@ -267,5 +267,5 @@
   <parent link="gripper-base_link"/>
   <child link="camera_frame"/>
-  <origin xyz="-0.17 0.033 -0.033" rpy="3.14159265 0 0"/>
+  <origin xyz="0.17 -0.033 -0.033" rpy="3.14159265 0 3.14159265"/>
 </joint>
 </xacro:macro>

File: ri_seaweed_ws/src/robot_description/kuka_agilus_support/urdf/kr10_r900_2.urdf.xacro (robot description, xacro)
@@ -38,5 +38,5 @@
   <xacro:gripper/>
   <joint name="flange-gripper-base_link" type="fixed">
-    <origin xyz="0 0 0" rpy="1.5708 0 -1.5708" />
+    <origin xyz="0 0 0" rpy="1.5708 3.14159265 -1.5708" />
     <parent link="flange" />
     <child link="gripper-base_link" />

Commit message: Extended the pickup test + small fixes

File: ri_seaweed_ws/src/robot_description/gripper_support/urdf/gripper.xacro (robot description, xacro)
@@ -267,5 +267,5 @@
   <parent link="gripper-base_link"/>
   <child link="camera_frame"/>
-  <origin xyz="0.17 -0.033 -0.033" rpy="3.14159265 0 3.14159265"/>
+  <origin xyz="0.205 -0.023 -0.033" rpy="3.14159265 0 3.14159265"/>
 </joint>
 </xacro:macro>

Commit message: Cleaned up the code and added more examples

File: ri_seaweed_ws/src/robot_description/gripper_support/urdf/gripper.xacro (robot description, xacro)
@@ -262,4 +262,10 @@
   <child link="claw_body_r_1"/>
 </joint>
+<link name="TCP"></link>
+<joint name="gripper-base_link_to_TCP_joint" type="fixed">
+  <parent link="gripper-base_link"/>
+  <child link="TCP"/>
+  <origin xyz="0 -0.04 -0.09" rpy="0 0 0"/>
+</joint>
 <!-- Transfer from camera to gripper base -->
 <link name="camera_frame"></link>
@@ -267,5 +273,5 @@
   <parent link="gripper-base_link"/>
   <child link="camera_frame"/>
-  <origin xyz="0.205 -0.023 -0.033" rpy="3.14159265 0 3.14159265"/>
+  <origin xyz="0.2 -0.035 -0.015" rpy="3.14159265 0 3.14159265"/>
 </joint>
 </xacro:macro>
